File: pcb/camera-clicker.kicad_sch (KiCad schematic)
At the start: 31 parts, among them J1 USB_C_Receptacle_USB2.0, SW2 BOOT, SW3 RST, SW4 SW_DPST_x2, SW5 SW_SPDT, U2 ESP32-MINI-1, U3 MCP2221AxST, U4 AZ1117-3.3

Commit message: first layout
Parts:
- removed SW5: SW_SPDT, switch-footprints:1825232-1_TEC, symbol Switch:SW_SPDT
- added J2: Conn_01x06, Connector_PinHeader_2.54mm:PinHeader_1x06_P2.54mm_Vertical, symbol Connector_Generic:Conn_01x06
- added SW1: SW_SPST, Button_Switch_THT:SW_CuK_OS102011MA1QN1_SPDT_Angled, symbol Switch:SW_SPDT
- SW4: footprint (none) -> CameraClickerFootprints:EVPAX-A1A
- TH1: footprint Resistor_SMD:R_0402_1005Metric -> Resistor_SMD:R_1206_3216Metric_Pad1.30x1.75mm_HandSolder
Connections:
- net +3.3V: now also J2.2 (Pin_2)
- net +5V: now also J2.1 (Pin_1)
- net +BATT: now also J2.3 (Pin_3), SW1.3 (C)
- net GND: now also U1.9 (THERM), J2.6 (Pin_6)
- net RX: now also J2.5 (Pin_5)
- net TX: now also J2.4 (Pin_4)
- net at BT1.1 (+), C2.1, R3.2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: now also SW1.2 (B)

Commit message: more pcb
Parts:
- added H1, H2, H3, H4: MountingHole, MountingHole:MountingHole_2.2mm_M2, symbol Mechanical:MountingHole
Connections:
- no-connect marks 32 -> 33
Changed lines of the file:
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@@
   (no_connect (at 43.18 82.55))
   (no_connect (at 109.22 77.47))
+  (no_connect (at -21.59 86.36))
   (no_connect (at 43.18 92.71))
   (no_connect (at 43.18 90.17))
@@
     )
   )
+  (symbol (lib_id "Mechanical:MountingHole") (at 35.56 186.69 0) (unit 1)
+    (in_bom yes) (on_board yes) (dnp no) (fields_autoplaced)
+    (property "Reference" "H2" (at 38.1 186.0463 0)
+      (effects (font (size 1.27 1.27)) (justify left))
+    )
+    (property "Value" "MountingHole" (at 38.1 187.9673 0)
+      (effects (font (size 1.27 1.27)) (justify left))
+    )
+    (property "Footprint" "MountingHole:MountingHole_2.2mm_M2" (at 35.56 186.69 0)
+      (effects (font (size 1.27 1.27)) hide)
+    )
+    (property "Datasheet" "~" (at 35.56 186.69 0)
+      (effects (font (size 1.27 1.27)) hide)
+    )
+    (instances
+      (project "camera-clicker"
+        (path "/0d623961-149c-4284-bf33-70ef9e2abb2a"
+          (reference "H2") (unit 1)
+        )
+      )
+    )
+  )
   (symbol (lib_id "Device:Thermistor_NTC") (at 255.27 53.34 180) (unit 1)
     (in_bom yes) (on_board yes) (dnp no) (fields_autoplaced)
@@
         (path "/0d623961-149c-4284-bf33-70ef9e2abb2a"
           (reference "TH1") (unit 1)
+        )
+      )
+    )
+  )
+  (symbol (lib_id "Mechanical:MountingHole") (at 27.94 186.69 0) (unit 1)
+    (in_bom yes) (on_board yes) (dnp no) (fields_autoplaced)
+    (property "Reference" "H1" (at 30.48 186.0463 0)
+      (effects (font (size 1.27 1.27)) (justify left))
+    )
+    (property "Value" "MountingHole" (at 30.48 187.9673 0)
+      (effects (font (size 1.27 1.27)) (justify left))
+    )
+    (property "Footprint" "MountingHole:MountingHole_2.2mm_M2" (at 27.94 186.69 0)
+      (effects (font (size 1.27 1.27)) hide)
+    )
+    (property "Datasheet" "~" (at 27.94 186.69 0)
+      (effects (font (size 1.27 1.27)) hide)
+    )
+    (instances
+      (project "camera-clicker"
+        (path "/0d623961-149c-4284-bf33-70ef9e2abb2a"
+          (reference "H1") (unit 1)
         )
       )
@@
     )
   )
+  (symbol (lib_id "Mechanical:MountingHole") (at 44.45 186.69 0) (unit 1)
+    (in_bom yes) (on_board yes) (dnp no) (fields_autoplaced)
+    (property "Reference" "H3" (at 46.99 186.0463 0)
+      (effects (font (size 1.27 1.27)) (justify left))
+    )
+    (property "Value" "MountingHole" (at 46.99 187.9673 0)
+      (effects (font (size 1.27 1.27)) (justify left))
+    )
+    (property "Footprint" "MountingHole:MountingHole_2.2mm_M2" (at 44.45 186.69 0)
+      (effects (font (size 1.27 1.27)) hide)
+    )
+    (property "Datasheet" "~" (at 44.45 186.69 0)
+      (effects (font (size 1.27 1.27)) hide)
+    )
+    (instances
+      (project "camera-clicker"
+        (path "/0d623961-149c-4284-bf33-70ef9e2abb2a"
+          (reference "H3") (unit 1)
+        )
+      )
+    )
+  )
   (symbol (lib_id "Switch:SW_SPST") (at 118.11 69.85 0) (unit 1)
     (in_bom yes) (on_board yes) (dnp no) (fields_autoplaced)
@@
         )
       )
+    )
+  )
+  (symbol (lib_id "Mechanical:MountingHole") (at 53.34 186.69 0) (unit 1)
+    (in_bom yes) (on_board yes) (dnp no) (fields_autoplaced)
+    (property "Reference" "H4" (at 55.88 186.0463 0)
+      (effects (font (size 1.27 1.27)) (justify left))
+    )
+    (property "Value" "MountingHole" (at 55.88 187.9673 0)
+      (effects (font (size 1.27 1.27)) (justify left))
+    )
+    (property "Footprint" "MountingHole:MountingHole_2.2mm_M2" (at 53.34 186.69 0)
+      (effects (font (size 1.27 1.27)) hide)
+    )
+    (property "Datasheet" "~" (at 53.34 186.69 0)
+      (effects (font (size 1.27 1.27)) hide)
+    )
+    (instances
+      (project "camera-clicker"
+        (path "/0d623961-149c-4284-bf33-70ef9e2abb2a"
+          (reference "H4") (unit 1)
+        )
+      )

Commit message: update pcb
Parts:
- U1: value ~ -> BQ25170
Changed lines of the file:
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@@
   (symbol (lib_id "CameraClickerLibrary:BQ25170DSGR") (at 231.14 43.18 0) (unit 1)
     (in_bom yes) (on_board yes) (dnp no) (fields_autoplaced)
-    (property "Reference" "U1" (at 231.14 34.5981 0)
+    (property "Reference" "U1" (at 231.14 32.6771 0)
       (effects (font (size 1.27 1.27)))
     )
-    (property "Value" "~" (at 231.14 43.18 0)
+    (property "Value" "BQ25170" (at 231.14 34.5981 0)
       (effects (font (size 1.27 1.27)))
     )

Commit message: update pcb
Parts:
- removed C3: 22uf, Capacitor_SMD:C_1206_3216Metric, symbol Device:C
- removed C4: 10uf, Capacitor_SMD:C_1206_3216Metric, symbol Device:C
- removed C5: 0.47uf, Capacitor_SMD:C_1206_3216Metric, symbol Device:C
- removed R9: 10k, Resistor_SMD:R_1206_3216Metric, symbol Device:R_US
- removed U3: MCP2221AxST, Package_SO:TSSOP-14_4.4x5mm_P0.65mm, symbol Interface_USB:MCP2221AxST
- removed U4: AZ1117-3.3, Package_TO_SOT_SMD:SOT-89-3, symbol Regulator_Linear:AZ1117-3.3
Connections:
- net D+: no longer names the net of J1.A6 (D+)
- net D+: no longer J1.B6 (D+)
- net D-: no longer names the net of J1.A7 (D-)
- net D-: no longer J1.B7 (D-)
- no-connect marks 33 -> 31

Commit message: new pcb design
Parts:
- removed J1: USB_C_Receptacle_USB2.0, Connector_USB:USB_C_Receptacle_GCT_USB4085, symbol Connector:USB_C_Receptacle_USB2.0
- added J3: USB_C_Receptacle_PowerOnly_6P, switch-footprints:USB_C_Receptacle_Amphenol_10164359-3A, symbol Connector:USB_C_Receptacle_PowerOnly_6P
- SW2, SW3: footprint Button_Switch_THT:SW_PUSH_6mm -> switch-footprints:SW_SPST_PTS526
Connections:
- net +3.3V is gone; now on net +BATT: J2.2 (Pin_2)
- net +5V: now also J3.A9 (VBUS), J3.B9 (VBUS)
- net GND: now also J3.A12 (GND), J3.B12 (GND), J3.S1 (SHIELD)
- net at R8.1: now also J3.A5 (CC1)
- net at R7.1: now also J3.B5 (CC2)
- no-connect marks 31 -> 25
Other:
- moved on the sheet: R7, R8

Commit message: updating pcb
Other:
- title: (none) -> Camera Clicker
Changed lines of the file:
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@@
 (kicad_sch (version 20230121) (generator eeschema)
   (paper "A4")
+  (title_block
+    (title "Camera Clicker")
+    (comment 1 "Olympus OM-D Cameras with WiFi")
+    (comment 2 "Apache-2.0 License")
+    (comment 3 "© Aaron Patterson")
+  )
   (junction (at 86.36 52.07) (diameter 0) (color 0 0 0 0)
   )

Commit message: updates
Parts:
- BT1: Link (none) -> https://www.digikey.com/en/products/detail/keystone-electro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
- J3: Link (none) -> https://www.digikey.com/en/products/detail/amphenol-cs-fci/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
- SW1: Link (none) -> https://www.digikey.com/en/products/detail/te-connectivity-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
- SW2, SW3: Link (none) -> https://www.digikey.com/en/products/detail/c-k/PTS526-SK15-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
- SW4: Link (none) -> https://www.digikey.com/en/products/detail/panasonic-electr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
- U1: Link (none) -> https://www.digikey.com/en/products/detail/texas-instrument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
- U2: Link (none) -> https://www.digikey.com/en/products/detail/espressif-system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
Changed lines of the file:
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@@
+      (effects (font (size 1.27 1.27)) hide)
+    )
+    (property "Link" "https://www.digikey.com/en/products/detail/amphenol-cs-fci/10164359-00011LF/18443702" (at 233.68 96.52 0)
       (effects (font (size 1.27 1.27)) hide)
     )
@@
       (effects (font (size 1.27 1.27)) hide)
     )
-    (property "Datasheet" "~" (at 77.47 154.94 0)
+    (property "Datasheet" "https://www3.panasonic.biz/ac/e_download/control/switch/light-touch/catalog/sw_lt_eng_3026s_w.pdf" (at 77.47 154.94 0)
+      (effects (font (size 1.27 1.27)) hide)
+    )
+    (property "Link" "https://www.digikey.com/en/products/detail/panasonic-electronic-components/EVP-AXBA1A/4930566" (at 77.47 154.94 0)
       (effects (font (size 1.27 1.27)) hide)
     )
@@
       (effects (font (size 1.27 1.27)) hide)
     )
+    (property "Link" "https://www.digikey.com/en/products/detail/te-connectivity-alcoswitch-switches/1825232-1/4021554" (at 264.16 31.75 90)
+      (effects (font (size 1.27 1.27)) hide)
+    )
     (pin "1")
     (pin "2")
@@
       (effects (font (size 1.27 1.27)) hide)
     )
-    (property "Datasheet" "~" (at 34.29 62.23 0)
+    (property "Datasheet" "https://www.ckswitches.com/media/2780/pts526.pdf" (at 34.29 62.23 0)
+      (effects (font (size 1.27 1.27)) hide)
+    )
+    (property "Link" "https://www.digikey.com/en/products/detail/c-k/PTS526-SK15-SMTR2-LFS/10056626" (at 34.29 62.23 0)
       (effects (font (size 1.27 1.27)) hide)
     )
@@
       (effects (font (size 1.27 1.27)) hide)
     )
-    (property "Datasheet" "~" (at 118.11 69.85 0)
+    (property "Datasheet" "https://www.ckswitches.com/media/2780/pts526.pdf" (at 118.11 69.85 0)
+      (effects (font (size 1.27 1.27)) hide)
+    )
+    (property "Link" "https://www.digikey.com/en/products/detail/c-k/PTS526-SK15-SMTR2-LFS/10056626" (at 118.11 69.85 0)
       (effects (font (size 1.27 1.27)) hide)
     )
@@
     )
     (property "Datasheet" "https://www.espressif.com/sites/default/files/documentation/esp32-mini-1_datasheet_en.pdf" (at 76.2 143.51 0)
+      (effects (font (size 1.27 1.27)) hide)
+    )
+    (property "Link" "https://www.digikey.com/en/products/detail/espressif-systems/ESP32-MINI-1-N4/13532111" (at 76.2 87.63 0)
       (effects (font (size 1.27 1.27)) hide)
     )
@@
       (effects (font (size 1.27 1.27)) hide)
     )
-    (property "Datasheet" "~" (at 264.16 40.386 90)
+    (property "Datasheet" "https://www.keyelco.com/userAssets/file/M65p27.pdf" (at 264.16 40.386 90)
+      (effects (font (size 1.27 1.27)) hide)
+    )
+    (property "Link" "https://www.digikey.com/en/products/detail/keystone-electronics/1042/2745668" (at 264.16 41.91 0)
       (effects (font (size 1.27 1.27)) hide)
     )
@@
       (effects (font (size 1.27 1.27)) hide)
     )
-    (property "Datasheet" "~" (at 77.47 146.05 0)
+    (property "Datasheet" "https://www3.panasonic.biz/ac/e_download/control/switch/light-touch/catalog/sw_lt_eng_3026s_w.pdf" (at 77.47 146.05 0)
+      (effects (font (size 1.27 1.27)) hide)
+    )
+    (property "Link" "https://www.digikey.com/en/products/detail/panasonic-electronic-components/EVP-AXBA1A/4930566" (at 77.47 146.05 0)
       (effects (font (size 1.27 1.27)) hide)
     )
@@
       (effects (font (size 1.27 1.27)) hide)
     )
+    (property "Link" "https://www.digikey.com/en/products/detail/texas-instruments/BQ25170DSGR/14124032" (at 231.14 43.18 0)
+      (effects (font (size 1.27 1.27)) hide)
+    )
